File: Hardware/PCB-PCFB-001/Schematics/pcb-pcfb-001/pcb-pcfb-001.kicad_sch (KiCad schematic)
At the start: 58 parts, among them J1 Fan1, J10 5Volts 10Amp, J11 RPI4-#1_PWR, J12 RPI4-#2_PWR, J13 RPI4-#3_PWR, J14 RPI4-#4_PWR, J2 Fan2, J3 Fan3, J4 Fan4, J5 RPI4-FAN1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

Commit message: updating
Parts:
- removed C1, C3: 1000uF, symbol Device:C_Polarized
- removed C2, C4, C5, C6: 1uF, symbol Device:C_Polarized
- removed J1: Fan1, symbol Connector_Generic:Conn_01x02
- removed J10: 5Volts 10Amp, symbol Connector_Generic:Conn_01x02
- removed J11: RPI4-#1_PWR, symbol Connector_Generic:Conn_01x02
- removed J12: RPI4-#2_PWR, symbol Connector_Generic:Conn_01x02
- removed J13: RPI4-#3_PWR, symbol Connector_Generic:Conn_01x02
- removed J14: RPI4-#4_PWR, symbol Connector_Generic:Conn_01x02
- removed J2: Fan2, symbol Connector_Generic:Conn_01x02
- removed J3: Fan3, symbol Connector_Generic:Conn_01x02
- removed J4: Fan4, symbol Connector_Generic:Conn_01x02
- removed J5: RPI4-FAN1, symbol Connector_Generic:Conn_01x02
- removed J6: RPI4-FAN2, symbol Connector_Generic:Conn_01x02
- removed J7: RPI4-FAN3, symbol Connector_Generic:Conn_01x02
- removed J8: RPI4-FAN4, symbol Connector_Generic:Conn_01x02
- removed J9: 12Volts, symbol Connector:Barrel_Jack_Switch
- removed M1: Fan1, symbol Motor:Fan_ALT
- removed M2: Fan2, symbol Motor:Fan_ALT
- removed M3: Fan3, symbol Motor:Fan_ALT
- removed M4: Fan4, symbol Motor:Fan_ALT
- removed Q1, Q2, Q3, Q4: NPN, symbol Simulation_SPICE:NPN
- removed R1: 1k, symbol Device:R
- removed R10, R3, R4, R5, R6, R7, R8, R9: R, symbol Device:R
- removed R11, R12, R18, R19, R21, R23, R24, R25: 1K, symbol Device:R
- removed R13, R14, R15, R16, R17, R20, R22, R26: 62K, symbol Device:R
- removed R2: 220R, symbol Device:R
- removed U1: LM317_TO-220, Package_TO_SOT_THT:TO-220-3_Vertical, symbol Regulator_Linear:LM317_TO-220
- removed U2, U3: LM358, symbol Amplifier_Operational:LM358
- removed U4: MAX232, symbol Interface_UART:MAX232
Other:
- added sheet Distribuição energia (distribuicao_energia.kicad_sch)
- added sheet Placa Controle Fans (placaControleFans.kicad_sch)
- added sheet Placa de leds (placadeleds.kicad_sch)
- note removed: "não foi implementado nos teste em protoboard funcionou corretamente porém nessa placa não funcionou, apesar que nos resistores de entrada aparecia igual nos testes 48mA, porem a saida fica em -7.0v"
